File: project4_pcb/_autosave-PWMGenerator-mhe4.kicad_sch (KiCad schematic)
At the start: 30 parts, among them J1 Conn_01x03_Pin, Q1 2N3904, Q2 2N3904, Q3 2N3906, Q4 2N3906, SW1 SW_SPST, U1 LM7805_TO220, U2 LM339

Commit message: all error fixed
1
Connections:
- net GND: now also U2.12 (V-)
- net at C2.1, J1.1 (Pin_1), Q4.3 (C)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: now also U2.3 (V+)
- no-connect marks 0 -> 9
