File: project4_pcb/PWMGenerator-mhe4.kicad_sch (KiCad schematic)
At the start: 30 parts, among them J1 Conn_01x03_Pin, Q1 2N3904, Q2 2N3904, Q3 2N3906, Q4 2N3906, SW1 SW_SPST, U1 LM7805_TO220, U2 LM339

Commit message: partB still working
1
Parts:
- added unit 1 of U2
- added unit 3 of U2
- added unit 4 of U2
- added unit 2 of U2
- C3: footprint (none) -> Capacitor_SMD:C_0805_2012Metric
- D1, D2, D3, D4, D5: value 1N4005 -> 1N4005G; footprint Diode_THT:D_DO-41_SOD81_P10.16mm_Horizontal -> Diode_SMD:D_0805_2012Metric
- D6: value LED -> LED_GREEN; footprint (none) -> LED_THT:LED_D5.0mm_GREEN
- Q1, Q2, Q3, Q4: footprint Package_TO_SOT_THT:TO-92_Inline -> Package_TO_SOT_SMD:SOT-23
- R1, R10, R11, R2, R3, R4, R5, R6, R7, R8: footprint (none) -> Resistor_SMD:R_0805_2012Metric
- U2: footprint (none) -> Package_SO:SOIC-14_3.9x8.7mm_P1.27mm
Connections:
- net GND: now also U2.12 (V-)
- net at C2.1, J1.1 (Pin_1), Q4.3 (C)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: now also U2.3 (V+)
- net at R10.1: now also U2.2; no longer U2.2
- net at C3.1, Q2.3 (C), Q3.1 (E): now also U2.4 (-); no longer U2.4 (-)
- net at R8.2, RV1.1: now also U2.5 (+); no longer U2.5 (+)
- no-connect marks 0 -> 9
