File: project4_pcb/PWMGenerator-mhe4.kicad_sch (KiCad schematic)
At the start: 30 parts, among them J1 Conn_01x03_Pin, Q1 2N3904, Q2 2N3904, Q3 2N3906, Q4 2N3906, SW1 SW_SPST, U1 LM7805_TO220, U2 LM339

Commit message: setting update
1
Parts:
- C1: footprint (none) -> Capacitor_THT:CP_Radial_D8.0mm_P3.50mm
- C2: footprint (none) -> Capacitor_THT:CP_Radial_D4.0mm_P1.50mm
- RV1: footprint (none) -> Potentiometer_THT:Potentiometer_Alps_RK09K_Single_Vertical
- SW1: value SW_SPST -> CTS 209-210; footprint (none) -> Button_Switch_THT:SW_DIP_SPSTx01_Slide_6.7x4.1mm_W7.62mm_P2.54mm_LowProfile
- V1: footprint (none) -> Connector_BarrelJack:BarrelJack_Horizontal; symbol Simulation_SPICE:VSIN -> Connector:Barrel_Jack
Changed lines of the file:
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@@
 		(title "CMPE2150 PWM Generator - mhe4")
 		(date "2025-12-11")
-		(rev "0")
+		(rev "2")
 		(company "NAIT CNT")
 		(comment 1 "Mengning He")
@@
 	(wire
 		(pts
+			(xy 31.75 44.45) (xy 31.75 52.07)
+		)
+		(stroke
+			(width 0)
+			(type default)
+		)
+	)
+	(wire
+		(pts
 			(xy 78.74 34.29) (xy 82.55 34.29)
 		)
@@
 	(wire
 		(pts
-			(xy 31.75 59.69) (xy 31.75 77.47)
+			(xy 31.75 57.15) (xy 31.75 77.47)
 		)
 		(stroke
@@
 	(wire
 		(pts
-			(xy 31.75 44.45) (xy 31.75 49.53)
-		)
-		(stroke
-			(width 0)
-			(type default)
-		)
-	)
-	(wire
-		(pts
 			(xy 68.58 60.96) (xy 68.58 63.5)
 		)
@@
 			)
 		)
-		(property "Footprint" ""
+		(property "Footprint" "Capacitor_THT:CP_Radial_D4.0mm_P1.50mm"
 			(at 110.1852 45.72 0)
 			(effects
@@
 			)
 		)
-		(property "Datasheet" "~"
+		(property "Datasheet" "https://industrial.panasonic.com/cdbs/www-data/pdf/RDF0000/ABA0000C1059.pdf"
 			(at 109.22 41.91 0)
 			(effects
@@
 			)
 		)
-		(property "Value" "SW_SPST"
+		(property "Value" "CTS 209-210"
 			(at 27.94 39.37 0)
 			(effects
@@
 			)
 		)
-		(property "Footprint" ""
+		(property "Footprint" "Button_Switch_THT:SW_DIP_SPSTx01_Slide_6.7x4.1mm_W7.62mm_P2.54mm_LowProfile"
 			(at 31.75 39.37 0)
 			(effects
@@
 			)
 		)
-		(property "Datasheet" "~"
+		(property "Datasheet" "https://www.ctscorp.com/wp-content/uploads/209-210.pdf"
 			(at 31.75 39.37 0)
 			(effects
@@
 		(dnp no)
 		(property "Reference" "RV1"
-			(at 183.134 64.008 0)
+			(at 180.594 64.262 0)
 			(effects
 				(font
@@
 		)
 		(property "Value" "5k"
-			(at 183.134 61.468 0)
+			(at 180.594 61.722 0)
 			(effects
 				(font
@@
 			)
 		)
-		(property "Footprint" ""
+		(property "Footprint" "Potentiometer_THT:Potentiometer_Alps_RK09K_Single_Vertical"
 			(at 176.53 62.23 0)
 			(effects
@@
 			)
 		)
-		(property "Datasheet" "~"
+		(property "Datasheet" "https://tech.alpsalpine.com/prod/e/pdf/potentiometer/rotarypotentiometers/rk09k/rk09k.pdf"
 			(at 176.53 62.23 0)
 			(effects
@@
 	)
 	(symbol
-		(lib_id "Simulation_SPICE:VSIN")
-		(at 31.75 54.61 0)
+		(lib_id "Connector:Barrel_Jack")
+		(at 24.13 54.61 0)
 		(unit 1)
 		(exclude_from_sim no)
@@
 		(dnp no)
 		(property "Reference" "V1"
-			(at 23.114 54.864 0)
+			(at 19.812 46.482 0)
 			(effects
 				(font
@@
 		)
 		(property "Value" "VSIN"
-			(at 23.114 57.404 0)
+			(at 19.812 49.022 0)
 			(effects
 				(font
@@
 			)
 		)
-		(property "Footprint" ""
-			(at 31.75 54.61 0)
+		(property "Footprint" "Connector_BarrelJack:BarrelJack_Horizontal"
+			(at 25.4 55.626 0)
 			(effects
 				(font
@@
 			)
 		)
-		(property "Datasheet" "https://ngspice.sourceforge.io/docs/ngspice-html-manual/manual.xhtml#sec_Independent_Sources_for"
-			(at 31.75 54.61 0)
+		(property "Datasheet" "~"
+			(at 25.4 55.626 0)
 			(effects
 				(font
@@
 			)
 		)
-		(property "Description" "Voltage source, sinusoidal"
-			(at 31.75 54.61 0)
+		(property "Description" "DC Barrel Jack"
+			(at 24.13 54.61 0)
 			(effects
 				(font
@@
 		)
 		(property "Sim.Pins" "1=+ 2=-"
-			(at 31.75 54.61 0)
+			(at 24.13 54.61 0)
 			(effects
 				(font
@@
 		)
 		(property "Sim.Params" "dc=0 ampl=16.97 f=60 ac=12"
-			(at 20.32 74.676 90)
+			(at 16.51 70.612 90)
 			(effects
 				(font
@@
 		)
 		(property "Sim.Type" "SIN"
-			(at 31.75 54.61 0)
+			(at 24.13 54.61 0)
 			(effects
 				(font
@@
 		)
 		(property "Sim.Device" "V"
-			(at 31.75 54.61 0)
+			(at 24.13 54.61 0)
 			(effects
 				(font
@@
 			)
 		)
-		(property "Footprint" ""
+		(property "Footprint" "Capacitor_THT:CP_Radial_D8.0mm_P3.50mm"
 			(at 83.5152 46.99 0)
 			(effects
@@
 			)
 		)
-		(property "Datasheet" "~"
+		(property "Datasheet" "https://www.nichicon.com/getmedia/8feec43d-7806-4ea3-a7e2-8f52c40026b3/e-upw.pdf"
 			(at 82.55 43.18 0)
 			(effects

Commit message: final schematic check(no error)
1
Parts:
- V1: value VSIN -> BarrelJack; footprint Connector_BarrelJack:BarrelJack_Horizontal -> Connector_BarrelJack:BarrelJack_SwitchcraftConxall_RAPC10U_Horizontal
Changed lines of the file:
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@@
 			)
 		)
-		(property "Value" "VSIN"
+		(property "Value" "BarrelJack"
 			(at 19.812 49.022 0)
 			(effects
@@
 			)
 		)
-		(property "Footprint" "Connector_BarrelJack:BarrelJack_Horizontal"
+		(property "Footprint" "Connector_BarrelJack:BarrelJack_SwitchcraftConxall_RAPC10U_Horizontal"
 			(at 25.4 55.626 0)
 			(effects
@@
 			)
 		)
-		(property "Datasheet" "~"
+		(property "Datasheet" "https://www.switchcraft.com/Drawings/RAPC10U_CD.pdf"
 			(at 25.4 55.626 0)
 			(effects
