File: project4_pcb/PWMGenerator-mhe4.kicad_sch (KiCad schematic)
At the start: 30 parts, among them J1 Conn_01x03_Pin, Q1 2N3904, Q2 2N3904, Q3 2N3906, Q4 2N3906, SW1 CTS 209-210, U1 LM7805_TO220, U2 LM339

Commit message: fix: potentiometer
1
Parts:
- RV1: symbol Device:R_Variable_US -> Device:R_Potentiometer_US
Connections:
- net GND: now also RV1.3
Changed lines of the file:
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@@
 		(title "CMPE2150 PWM Generator - mhe4")
 		(date "2025-12-11")
-		(rev "3")
+		(rev "5")
 		(company "NAIT CNT")
 		(comment 1 "Mengning He")
@@
 	)
 	(junction
-		(at 176.53 46.99)
-		(diameter 0)
-		(color 0 0 0 0)
-	)
-	(junction
 		(at 218.44 34.29)
 		(diameter 0)
@@
 	)
 	(junction
+		(at 176.53 46.99)
+		(diameter 0)
+		(color 0 0 0 0)
+	)
+	(junction
 		(at 163.83 58.42)
 		(diameter 0)
@@
 	)
 	(junction
+		(at 176.53 68.58)
+		(diameter 0)
+		(color 0 0 0 0)
+	)
+	(junction
 		(at 63.5 50.8)
 		(diameter 0)
@@
 	(wire
 		(pts
-			(xy 176.53 66.04) (xy 176.53 74.93)
-		)
-		(stroke
-			(width 0)
-			(type default)
-		)
-	)
-	(wire
-		(pts
 			(xy 82.55 83.82) (xy 76.2 83.82)
 		)
@@
 	(wire
 		(pts
+			(xy 176.53 66.04) (xy 176.53 68.58)
+		)
+		(stroke
+			(width 0)
+			(type default)
+		)
+	)
+	(wire
+		(pts
 			(xy 218.44 54.61) (xy 218.44 58.42)
 		)
@@
 	(wire
 		(pts
-			(xy 176.53 74.93) (xy 196.85 74.93)
+			(xy 34.29 29.21) (xy 38.1 29.21)
 		)
 		(stroke
@@
 	(wire
 		(pts
-			(xy 34.29 29.21) (xy 38.1 29.21)
+			(xy 238.76 74.93) (xy 218.44 74.93)
 		)
 		(stroke
@@
 	(wire
 		(pts
-			(xy 238.76 74.93) (xy 218.44 74.93)
+			(xy 44.45 50.8) (xy 39.37 50.8)
 		)
 		(stroke
@@
 	(wire
 		(pts
-			(xy 44.45 50.8) (xy 39.37 50.8)
+			(xy 95.25 46.99) (xy 95.25 49.53)
 		)
 		(stroke
@@
 	(wire
 		(pts
-			(xy 95.25 46.99) (xy 95.25 49.53)
+			(xy 44.45 72.39) (xy 54.61 72.39)
 		)
 		(stroke
@@
 	(wire
 		(pts
-			(xy 44.45 72.39) (xy 54.61 72.39)
+			(xy 171.45 68.58) (xy 176.53 68.58)
 		)
 		(stroke
@@
 	(wire
 		(pts
+			(xy 171.45 62.23) (xy 171.45 68.58)
+		)
+		(stroke
+			(width 0)
+			(type default)
+		)
+	)
+	(wire
+		(pts
 			(xy 196.85 34.29) (xy 218.44 34.29)
 		)
@@
 	(wire
 		(pts
+			(xy 176.53 68.58) (xy 176.53 74.93)
+		)
+		(stroke
+			(width 0)
+			(type default)
+		)
+	)
+	(wire
+		(pts
 			(xy 198.12 49.53) (xy 200.66 49.53)
 		)
@@
 	(wire
 		(pts
+			(xy 176.53 74.93) (xy 196.85 74.93)
+		)
+		(stroke
+			(width 0)
+			(type default)
+		)
+	)
+	(wire
+		(pts
 			(xy 238.76 41.91) (xy 238.76 74.93)
 		)
@@
 	(wire
 		(pts
+			(xy 176.53 46.99) (xy 176.53 58.42)
+		)
+		(stroke
+			(width 0)
+			(type default)
+		)
+	)
+	(wire
+		(pts
 			(xy 107.95 74.93) (xy 76.2 74.93)
 		)
@@
 	(wire
 		(pts
-			(xy 134.62 34.29) (xy 149.86 34.29)
+			(xy 172.72 62.23) (xy 171.45 62.23)
 		)
 		(stroke
@@
 	(wire
 		(pts
-			(xy 63.5 31.75) (xy 63.5 36.83)
+			(xy 134.62 34.29) (xy 149.86 34.29)
 		)
 		(stroke
@@
 	(wire
 		(pts
-			(xy 176.53 46.99) (xy 176.53 58.42)
+			(xy 63.5 31.75) (xy 63.5 36.83)
 		)
 		(stroke
@@
 	)
 	(symbol
-		(lib_id "Device:R_Variable_US")
+		(lib_id "Device:R_Potentiometer_US")
 		(at 176.53 62.23 0)
+		(mirror y)
 		(unit 1)
 		(exclude_from_sim no)
@@
 		(dnp no)
 		(property "Reference" "RV1"
-			(at 180.594 64.262 0)
+			(at 182.118 64.008 0)
 			(effects
 				(font
@@
 		)
 		(property "Value" "5k"
-			(at 180.594 61.722 0)
+			(at 181.102 61.214 0)
 			(effects
 				(font
@@
 			)
 		)
-		(property "Datasheet" "https://tech.alpsalpine.com/prod/e/pdf/potentiometer/rotarypotentiometers/rk09k/rk09k.pdf"
+		(property "Datasheet" "~"
 			(at 176.53 62.23 0)
 			(effects
@@
 			)
 		)
-		(property "Description" "Potentiometer"
+		(property "Description" "Potentiometer, US symbol"
 			(at 176.53 62.23 0)
 			(effects
@@
 		(pin "2"
 		)
+		(pin "3"
+		)
 		(instances
