File: project4_pcb/PWMGenerator-mhe4.kicad_pcb (KiCad board)
At the start: 2 copper layers, 0 parts

Commit message: ProjC_import success
1
Parts:
- added C1: 220uf, Capacitor_THT:CP_Radial_D8.0mm_P3.50mm, F.Cu at (74.3, -22.0)
- added C2: 10uf, Capacitor_THT:CP_Radial_D4.0mm_P1.50mm, F.Cu at (82.9, -24.0)
- added C3: 0.1uf, Capacitor_SMD:C_0805_2012Metric, F.Cu at (109.7, -49.0)
- added D1: 1N4005G, Diode_SMD:D_0805_2012Metric, F.Cu at (88.8, -39.6)
- added D2: 1N4005G, Diode_SMD:D_0805_2012Metric, F.Cu at (88.8, -36.5)
- added D3: 1N4005G, Diode_SMD:D_0805_2012Metric, F.Cu at (88.8, -33.5)
- added D4: 1N4005G, Diode_SMD:D_0805_2012Metric, F.Cu at (88.8, -30.5)
- added D5: 1N4005G, Diode_SMD:D_0805_2012Metric, F.Cu at (88.8, -27.4)
- added D6: LED_GREEN, LED_THT:LED_D5.0mm, F.Cu at (93.5, -22.6)
- added F1: NANOSMDC016F-2, lib:RESC3115X65N, F.Cu at (83.6, -19.5)
- added J1: Conn_01x03_Pin, Connector_PinHeader_2.54mm:PinHeader_1x03_P2.54mm_Vertical, F.Cu at (109.8, -57.9)
- added Q1: 2N3904, Package_TO_SOT_SMD:SOT-23, F.Cu at (105.1, -58.0)
- added Q2: 2N3904, Package_TO_SOT_SMD:SOT-23, F.Cu at (105.1, -53.5)
- added Q3: 2N3906, Package_TO_SOT_SMD:SOT-23, F.Cu at (105.1, -49.1)
- added Q4: 2N3906, Package_TO_SOT_SMD:SOT-23, F.Cu at (105.1, -44.6)
- added R1: 2.2k, Resistor_SMD:R_0805_2012Metric, F.Cu at (93.2, -39.6)
- added R10: 8.2k, Resistor_SMD:R_0805_2012Metric, F.Cu at (97.6, -30.8)
- added R11: 180, Resistor_SMD:R_0805_2012Metric, F.Cu at (97.6, -27.8)
- added R2: 1M, Resistor_SMD:R_0805_2012Metric, F.Cu at (93.2, -36.7)
- added R3: 330, Resistor_SMD:R_0805_2012Metric, F.Cu at (93.2, -33.7)
- added R4: 10k, Resistor_SMD:R_0805_2012Metric, F.Cu at (93.2, -30.8)
- added R5: 220k, Resistor_SMD:R_0805_2012Metric, F.Cu at (93.2, -27.8)
- added R6: 390k, Resistor_SMD:R_0805_2012Metric, F.Cu at (97.6, -39.6)
- added R7: 22k, Resistor_SMD:R_0805_2012Metric, F.Cu at (97.6, -36.7)
- added R8: 2.2k, Resistor_SMD:R_0805_2012Metric, F.Cu at (97.6, -33.7)
- added RV1: 5k, Potentiometer_THT:Potentiometer_Alps_RK09K_Single_Vertical, F.Cu at (72.8, -36.4)
- added SW1: CTS 209-210, Button_Switch_THT:SW_DIP_SPSTx01_Slide_6.7x4.1mm_W7.62mm_P2.54mm_LowProfile, F.Cu at (101.4, -32.2)
- added U1: LM7805_TO220, Package_TO_SOT_THT:TO-220-3_Vertical, F.Cu at (103.1, -37.2)
- added U2: LM339, Package_SO:SOIC-14_3.9x8.7mm_P1.27mm, F.Cu at (104.1, -24.1)
- added V1: BarrelJack, Connector_BarrelJack:BarrelJack_SwitchcraftConxall_RAPC10U_Horizontal, F.Cu at (100.6, -50.7)

Commit message: parct c cu
update
Parts:
- moved RV1 150.1 mm to (192.0, 54.8), turned to 180 degrees
- moved J1 146.7 mm to (186.4, 67.2)
- moved V1 139.2 mm to (76.2, 86.4)
- moved Q4 137.6 mm to (181.5, 69.8)
- moved R11 135.9 mm to (191.2, 70.8)
- moved Q1 124.0 mm to (141.0, 60.6)
- moved C3 119.1 mm to (170.3, 53.5)
- moved R10 115.9 mm to (170.1, 59.6)
- moved R2 115.3 mm to (135.1, 70.8)
- moved R8 114.8 mm to (151.4, 67.7)
- moved R1 110.9 mm to (134.9, 63.2)
- moved Q2 110.4 mm to (141.0, 50.9)
- moved Q3 109.8 mm to (152.5, 50.0)
- moved R7 109.0 mm to (155.0, 56.1)
- moved R6 108.1 mm to (147.9, 56.1)
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Routing:
- net Net-(SW1-A): track 0.00 -> 25.9 mm
- added copper zone on B.Cu, net GND
- added copper zone on F.Cu, net VCC
Other:
- board outline added: 154.4 x 64.5 mm
